File: FtdiTranslator.sch (KiCad schematic (older format))
At the start: 17 parts, among them P1 FTDI-DEVICE, P2 FTDI-HOST, Q1 2N7000, Q2 2N7000, Q3 2N7000, U1 MCP1700

Commit message: Update to Kicad 5
Parts:
- C1, C2: symbol C -> Device:C
- JP1, JP2, JP3: symbol Jumper_NO_Small -> Device:Jumper_NO_Small
- P1: symbol FTDI-DEVICE -> Components:FTDI-DEVICE
- P2: symbol FTDI-HOST -> Components:FTDI-HOST
- Q1, Q2, Q3: symbol 2N7000 -> Transistor_FET:2N7000
- R1, R2, R3, R4, R5, R6: symbol R -> Device:R
- U1: symbol MCP1700-3302E_SOT89 -> Regulator_Linear:MCP1700-3302E_SOT89
Changed lines of the file:
@@
-EESchema Schematic File Version 2
-LIBS:power
-LIBS:device
-LIBS:transistors
-LIBS:conn
-LIBS:linear
-LIBS:74xx
-LIBS:cmos4000
-LIBS:adc-dac
-LIBS:memory
-LIBS:xilinx
-LIBS:microcontrollers
-LIBS:dsp
-LIBS:microchip
-LIBS:analog_switches
-LIBS:motorola
-LIBS:texas
-LIBS:intel
-LIBS:audio
-LIBS:interface
-LIBS:digital-audio
-LIBS:philips
-LIBS:display
-LIBS:cypress
-LIBS:siliconi
-LIBS:opto
-LIBS:atmel
-LIBS:contrib
-LIBS:valves
-LIBS:Components
-LIBS:regul
+EESchema Schematic File Version 4
 LIBS:FtdiTranslator-cache
-EELAYER 25 0
+EELAYER 26 0
 EELAYER END
 $Descr User 8268 5846
@@
 $EndDescr
 $Comp
-L R R2
+L Device:R R2
 U 1 1 586288A4
 P 5850 950
@@
 $EndComp
 $Comp
-L R R1
+L Device:R R1
 U 1 1 586288DF
 P 5450 950
@@
 $EndComp
 $Comp
-L R R4
+L Device:R R4
 U 1 1 586294A6
 P 5150 1200
@@
 $EndComp
 $Comp
-L R R3
+L Device:R R3
 U 1 1 586294AC
 P 4750 1200
@@
 $EndComp
 $Comp
-L R R6
+L Device:R R6
 U 1 1 5862978D
 P 5800 1650
@@
 $EndComp
 $Comp
-L R R5
+L Device:R R5
 U 1 1 58629793
 P 5400 1650
@@
 NoConn ~ 6400 1650
 $Comp
-L GND #PWR01
+L power:GND #PWR01
 U 1 1 58642003
 P 4350 1750
@@
 $EndComp
 $Comp
-L GND #PWR02
+L power:GND #PWR02
 U 1 1 58642043
 P 6400 1750
@@
 $EndComp
 $Comp
-L Jumper_NO_Small JP3
+L Device:Jumper_NO_Small JP3
 U 1 1 586432D8
 P 5650 2550
@@
 $EndComp
 Wire Wire Line
-	5400 2550 5550 2550
+	5400 2550 5500 2550
 Wire Wire Line
 	5750 2550 5850 2550
 Wire Wire Line
-	4800 2550 4650 2550
+	4800 2550 4700 2550
 Text Label 4650 2550 2    60   ~ 0
 HV
@@
 LV
 $Comp
-L GND #PWR03
+L power:GND #PWR03
 U 1 1 586449A9
 P 5100 2950
@@
 $EndComp
 $Comp
-L FTDI-DEVICE P1
+L Components:FTDI-DEVICE P1
 U 1 1 595BABF7
 P 3950 1450
@@
 $EndComp
 $Comp
-L FTDI-HOST P2
+L Components:FTDI-HOST P2
 U 1 1 595BAF16
 P 6800 1450
@@
 LV
 $Comp
-L Jumper_NO_Small JP1
+L Device:Jumper_NO_Small JP1
 U 1 1 595C04F3
 P 4850 900
@@
 $EndComp
 $Comp
-L Jumper_NO_Small JP2
+L Device:Jumper_NO_Small JP2
 U 1 1 595C0569
 P 6200 1250
@@
 	5650 800  5850 800
 $Comp
-L 2N7000 Q2
+L Transistor_FET:2N7000 Q2
 U 1 1 595C9FF8
 P 4950 1250
@@
 $EndComp
 $Comp
-L 2N7000 Q3
+L Transistor_FET:2N7000 Q3
 U 1 1 595CA05E
 P 5600 1700
@@
 	4950 1050 5150 1050
 $Comp
-L MCP1700-3302E_SOT89 U1
+L Regulator_Linear:MCP1700-3302E_SOT89 U1
 U 1 1 595E5DC0
 P 5100 2550
@@
 $EndComp
 Wire Wire Line
-	5100 2950 5100 2850
-$Comp
-L 2N7000 Q1
+	5100 2950 5100 2900
+$Comp
+L Transistor_FET:2N7000 Q1
 U 1 1 595C9D4B
 P 5650 1000
@@
 $EndComp
 $Comp
-L C C1
+L Device:C C1
 U 1 1 595EA12E
 P 4700 2750
@@
 $EndComp
 $Comp
-L C C2
+L Device:C C2
 U 1 1 595EA1FB
 P 5500 2750
@@
 Connection ~ 4700 2550
 Wire Wire Line
-	4700 2900 5500 2900
+	4700 2900 5100 2900
 Connection ~ 5100 2900
 $Comp
-L PWR_FLAG #FLG04
+L power:PWR_FLAG #FLG04
 U 1 1 595EC89B
 P 6650 2500
@@
 $EndComp
 $Comp
-L PWR_FLAG #FLG05
+L power:PWR_FLAG #FLG05
 U 1 1 595EC8E0
 P 6650 2750
@@
 $EndComp
 $Comp
-L PWR_FLAG #FLG06
+L power:PWR_FLAG #FLG06
 U 1 1 595EC91E
 P 6650 3000
@@
 LV
 $Comp
-L GND #PWR07
+L power:GND #PWR07
 U 1 1 595EC9FB
 P 6800 3000
@@
 Wire Wire Line
 	6650 2500 6800 2500
+Wire Wire Line
+	5500 2550 5550 2550
+Wire Wire Line
+	4700 2550 4650 2550
+Wire Wire Line
+	5100 2900 5100 2850
+Wire Wire Line
+	5100 2900 5500 2900
 $EndSCHEMATC
